Commit message: camera not working

File: urdf/turtlebot3_waffle_pi.gazebo.xacro (robot description, xacro)
@@ -135,5 +135,5 @@
   </gazebo>
 <!--link : https://www.raspberrypi.org/documentation/hardware/camera/-->
-  <gazebo reference="camera_rgb_frame">
+  <!-- <gazebo reference="camera_rgb_frame">
     <sensor type="camera" name="Pi Camera">
       <always_on>true</always_on>
@@ -166,4 +166,4 @@
       </plugin>
     </sensor>
-  </gazebo>
+  </gazebo> -->
 </robot>

File: urdf/turtlebot3_waffle_pi.urdf.xacro (robot description, xacro)
@@ -160,5 +160,5 @@
     </inertial>
   </link>
-  <joint name="camera_joint" type="fixed">
+  <!-- <joint name="camera_joint" type="fixed">
     <origin xyz="0.073 -0.011 0.084" rpy="0 0 0"/>
     <parent link="base_link"/>
@@ -172,6 +172,6 @@
       </geometry>
     </collision>
-  </link>
-  <joint name="camera_rgb_joint" type="fixed">
+  </link> -->
+  <!-- <joint name="camera_rgb_joint" type="fixed">
     <origin xyz="0.003 0.011 0.009" rpy="0 0 0"/>
     <parent link="camera_link"/>
@@ -184,4 +184,9 @@
     <child link="camera_rgb_optical_frame"/>
   </joint>
-  <link name="camera_rgb_optical_frame"/>
+  <link name="camera_rgb_optical_frame"/> -->
+  <!-- d435i frame definition can be found at https://github.com/IntelRealSense/librealsense/blob/master/doc/d435i.md -->
+  <xacro:include filename="$(find mai_sim)/urdf/_d435i.urdf.xacro"/>
+  <xacro:sensor_d435i parent="base_link" name="D435i_camera" topics_ns="D435i_camera">
+    <origin xyz="0.0 0.5 0.1" rpy="0.0 0.0 0.0"/>
+  </xacro:sensor_d435i>
 </robot>
