Commit message: rtabmap with rs

File: urdf/_d435i.urdf.xacro (robot description, xacro)
@@ -1,196 +1,17 @@
 <?xml version="1.0"?>
 <!--
-Aknolegment: This file was copied from the realsense repository of
-pal-robotics-forks( https://github.com/pal-robotics-forks/realsense/ ).
-and then modified.
 License: Apache 2.0. See LICENSE file in root directory.
-Copyright(c) 2017 Intel Corporation. All Rights Reserved
-This is the URDF model for the Intel RealSense 430 camera, in it's
+Copyright(c) 2020 Intel Corporation. All Rights Reserved
+This is the URDF model for the Intel RealSense 435i camera, in it's
 aluminum peripherial evaluation case.
 -->
 <robot name="sensor_d435i" xmlns:xacro="http://ros.org/wiki/xacro">
-  <!--File includes-->
-  <xacro:include filename="$(find mai_sim)/urdf/_d435i.gazebo.xacro"/>
-  <xacro:macro name="sensor_d435i" params="parent
-                                          name:=camera
-                                          topics_ns:=camera
-                                          visualize:=true
-                                          align_depth:=false
-                                          enable_pointCloud:=false
-                                          unite_imu_method:=false
-                                          accel_fps:=250
-                                          gyro_fps:=400
-                                          clip_distance:=-1.0
-                                          depth_width:=1280
-                                          depth_height:=720
-                                          depth_fps:=30
-                                          infra_width:=640
-                                          infra_height:=480
-                                          infra_fps:=30
-                                          color_width:=1920
-                                          color_height:=1080
-                                          color_fps:=30
-                                          *origin">
-    <xacro:property name="M_PI" value="3.1415926535897931"/>
-    <!-- The following values are approximate, and the camera node
-     publishing TF values with actual calibrated camera extrinsic values -->
-    <xacro:property name="d435i_cam_depth_to_left_ir_offset" value="0.0"/>
-    <xacro:property name="d435i_cam_depth_to_right_ir_offset" value="-0.050"/>
-    <xacro:property name="d435i_cam_depth_to_color_offset" value="0.015"/>
-    <!-- The following values model the aluminum peripherial case for the
-  	D435 camera, with the camera joint represented by the actual
-  	peripherial camera tripod mount -->
-    <xacro:property name="d435i_cam_width" value="0.090"/>
-    <xacro:property name="d435i_cam_height" value="0.025"/>
-    <xacro:property name="d435i_cam_depth" value="0.02505"/>
-    <xacro:property name="d435i_cam_mount_from_center_offset" value="0.0149"/>
-    <!-- The following offset is relative the the physical D435 camera peripherial
-  	camera tripod mount -->
-    <xacro:property name="d435i_cam_depth_px" value="${d435i_cam_mount_from_center_offset}"/>
-    <xacro:property name="d435i_cam_depth_py" value="0.0175"/>
-    <xacro:property name="d435i_cam_depth_pz" value="${d435i_cam_height/2}"/>
-    <material name="${name}_aluminum">
-	  <color rgba="0.5 0.5 0.5 1"/>
-    </material>
-    <!-- camera body, with origin at bottom screw mount -->
-    <joint name="${name}_joint" type="fixed">
-      <xacro:insert_block name="origin"/>
-      <parent link="${parent}"/>
-      <child link="${name}_bottom_screw_frame"/>
-    </joint>
-    <link name="${name}_bottom_screw_frame"/>
-    <joint name="${name}_link_joint" type="fixed">
-      <origin xyz="0 ${d435i_cam_depth_py} ${d435i_cam_depth_pz}" rpy="0 0 0"/>
-      <parent link="${name}_bottom_screw_frame"/>
-      <child link="${name}_link"/>
-    </joint>
-    <link name="${name}_link">
-      <visual>
-      <origin xyz="${d435i_cam_mount_from_center_offset} ${-d435i_cam_depth_py} 0" rpy="${M_PI/2} 0 ${M_PI/2}"/>
-        <geometry>
-          <!-- <box size="${d435i_cam_width} ${d435i_cam_height} ${d435i_cam_depth}"/> -->
-          <mesh filename="package://realsense2_description/meshes/d435.dae"/>
-          <!--<mesh filename="package://realsense2_description/meshes/d435/d435.dae"/>-->
-        </geometry>
-        <material name="${name}_aluminum"/>
-      </visual>
-      <collision>
-        <origin xyz="0 ${-d435i_cam_depth_py} 0" rpy="0 0 0"/>
-        <geometry>
-        <box size="${d435i_cam_depth} ${d435i_cam_width} ${d435i_cam_height}"/>
-        </geometry>
-      </collision>
-      <inertial>
-        <!-- The following are not reliable values, and should not be used for modeling -->
-        <mass value="0.564"/>
-        <origin xyz="0 0 0"/>
-        <inertia ixx="0.003881243" ixy="0.0" ixz="0.0" iyy="0.000498940" iyz="0.0" izz="0.003879257"/>
-      </inertial>
-    </link>
-    <!-- camera depth joints and links -->
-    <joint name="${name}_depth_joint" type="fixed">
-      <origin xyz="0 0 0" rpy="0 0 0"/>
-      <parent link="${name}_link"/>
-      <child link="${name}_depth_frame"/>
-    </joint>
-    <link name="${name}_depth_frame"/>
-    <joint name="${name}_depth_optical_joint" type="fixed">
-      <origin xyz="0 0 0" rpy="${-M_PI/2} 0 ${-M_PI/2}"/>
-      <parent link="${name}_depth_frame"/>
-      <child link="${name}_depth_optical_frame"/>
-    </joint>
-    <link name="${name}_depth_optical_frame"/>
-    <!-- camera left IR joints and links -->
-    <joint name="${name}_left_ir_joint" type="fixed">
-      <origin xyz="0 ${d435i_cam_depth_to_left_ir_offset} 0" rpy="0 0 0"/>
-      <parent link="${name}_depth_frame"/>
-      <child link="${name}_left_ir_frame"/>
-    </joint>
-    <link name="${name}_left_ir_frame"/>
-    <joint name="${name}_left_ir_optical_joint" type="fixed">
-      <origin xyz="0 0 0" rpy="${-M_PI/2} 0 ${-M_PI/2}"/>
-      <parent link="${name}_left_ir_frame"/>
-      <child link="${name}_left_ir_optical_frame"/>
-    </joint>
-    <link name="${name}_left_ir_optical_frame"/>
-    <!-- camera right IR joints and links -->
-    <joint name="${name}_right_ir_joint" type="fixed">
-      <origin xyz="0 ${d435i_cam_depth_to_right_ir_offset} 0" rpy="0 0 0"/>
-      <parent link="${name}_depth_frame"/>
-      <child link="${name}_right_ir_frame"/>
-    </joint>
-    <link name="${name}_right_ir_frame"/>
-    <joint name="${name}_right_ir_optical_joint" type="fixed">
-      <origin xyz="0 0 0" rpy="${-M_PI/2} 0 ${-M_PI/2}"/>
-      <parent link="${name}_right_ir_frame"/>
-      <child link="${name}_right_ir_optical_frame"/>
-    </joint>
-    <link name="${name}_right_ir_optical_frame"/>
-    <!-- camera color joints and links -->
-    <joint name="${name}_color_joint" type="fixed">
-      <origin xyz="0 ${d435i_cam_depth_to_color_offset} 0" rpy="0 0 0"/>
-      <parent link="${name}_depth_frame"/>
-      <child link="${name}_color_frame"/>
-    </joint>
-    <link name="${name}_color_frame"/>
-    <joint name="${name}_color_optical_joint" type="fixed">
-      <origin xyz="0 0 0" rpy="${-M_PI/2} 0 ${-M_PI/2}"/>
-      <parent link="${name}_color_frame"/>
-      <child link="${name}_color_optical_frame"/>
-    </joint>
-    <link name="${name}_color_optical_frame"/>
-    <!-- camera accel joints and links -->
-    <joint name="${name}_accel_joint" type="fixed">
-      <origin xyz="-0.00174 0.00552 0.0176" rpy="0 0 0"/>
-      <parent link="${name}_link"/>
-      <child link="${name}_accel_frame"/>
-    </joint>
-    <link name="${name}_accel_frame"/>
-    <joint name="${name}_accel_optical_joint" type="fixed">
-      <origin xyz="0 0 0" rpy="${-M_PI/2} 0 ${-M_PI/2}"/>
-      <parent link="${name}_accel_frame"/>
-      <child link="${name}_accel_optical_frame"/>
-    </joint>
-    <link name="${name}_accel_optical_frame"/>
-    <!-- camera gyro joints and links -->
-    <joint name="${name}_gyro_joint" type="fixed">
-      <origin xyz="-0.00174 0.00552 0.0176" rpy="0 0 0"/>
-      <parent link="${name}_link"/>
-      <child link="${name}_gyro_frame"/>
-    </joint>
-    <link name="${name}_gyro_frame"/>
-    <joint name="${name}_gyro_optical_joint" type="fixed">
-      <origin xyz="0 0 0" rpy="${-M_PI/2} 0 ${-M_PI/2}"/>
-      <parent link="${name}_gyro_frame"/>
-      <child link="${name}_gyro_optical_frame"/>
-    </joint>
-    <link name="${name}_gyro_optical_frame"/>
-    <!-- Realsense Gazebo Plugin -->
-    <xacro:gazebo_d435i camera_name="${name}"
-                        topics_ns="${topics_ns}"
-                        reference_link="${name}_link"
-                        depth_optical_frame="${name}_depth_optical_frame"
-                        depth_width="${depth_width}"
-                        depth_height="${depth_height}"
-                        depth_fps="${depth_fps}"
-                        color_optical_frame="${name}_color_optical_frame"
-                        color_width="${color_width}"
-                        color_height="${color_height}"
-                        color_fps="${color_fps}"
-                        infrared1_optical_frame="${name}_left_ir_optical_frame"
-                        infrared2_optical_frame="${name}_right_ir_optical_frame"
-                        infra_width="${infra_width}"
-                        infra_height="${infra_height}"
-                        infra_fps="${infra_fps}"
-                        accel_optical_frame="${name}_accel_optical_frame"
-                        gyro_optical_frame="${name}_gyro_optical_frame"
-                        accel_fps="${accel_fps}"
-                        gyro_fps="${gyro_fps}"
-                        enable_pointCloud="${enable_pointCloud}"
-                        unite_imu_method="${unite_imu_method}"
-                        clip_distance="${clip_distance}"
-                        align_depth="${align_depth}"
-                        visualize="${visualize}"
-    />
+  <xacro:include filename="$(find mai_sim)/urdf/_d435.urdf.xacro"/>
+  <xacro:include filename="$(find mai_sim)/urdf/_d435i_imu_modules.urdf.xacro"/>
+  <xacro:macro name="sensor_d435i" params="parent *origin name:=camera use_nominal_extrinsics:=false">
+    <xacro:sensor_d435 parent="${parent}" name="${name}" use_nominal_extrinsics="${use_nominal_extrinsics}">
+      <xacro:insert_block name="origin" />
+    </xacro:sensor_d435>
+    <xacro:d435i_imu_modules name="${name}" use_nominal_extrinsics="${use_nominal_extrinsics}"/>
   </xacro:macro>
 </robot>

Commit message: kobuki with realsense

File: urdf/_d435i.urdf.xacro (robot description, xacro)
@@ -1,17 +1,196 @@
 <?xml version="1.0"?>
 <!--
+Aknolegment: This file was copied from the realsense repository of
+pal-robotics-forks( https://github.com/pal-robotics-forks/realsense/ ).
+and then modified.
 License: Apache 2.0. See LICENSE file in root directory.
-Copyright(c) 2020 Intel Corporation. All Rights Reserved
-This is the URDF model for the Intel RealSense 435i camera, in it's
+Copyright(c) 2017 Intel Corporation. All Rights Reserved
+This is the URDF model for the Intel RealSense 430 camera, in it's
 aluminum peripherial evaluation case.
 -->
 <robot name="sensor_d435i" xmlns:xacro="http://ros.org/wiki/xacro">
-  <xacro:include filename="$(find mai_sim)/urdf/_d435.urdf.xacro"/>
-  <xacro:include filename="$(find mai_sim)/urdf/_d435i_imu_modules.urdf.xacro"/>
-  <xacro:macro name="sensor_d435i" params="parent *origin name:=camera use_nominal_extrinsics:=false">
-    <xacro:sensor_d435 parent="${parent}" name="${name}" use_nominal_extrinsics="${use_nominal_extrinsics}">
-      <xacro:insert_block name="origin" />
-    </xacro:sensor_d435>
-    <xacro:d435i_imu_modules name="${name}" use_nominal_extrinsics="${use_nominal_extrinsics}"/>
+  <!--File includes-->
+  <xacro:include filename="$(find mai_sim)/urdf/_d435i.gazebo.xacro"/>
+  <xacro:macro name="sensor_d435i" params="parent
+                                          name:=camera
+                                          topics_ns:=camera
+                                          visualize:=true
+                                          align_depth:=false
+                                          enable_pointCloud:=false
+                                          unite_imu_method:=false
+                                          accel_fps:=250
+                                          gyro_fps:=400
+                                          clip_distance:=-1.0
+                                          depth_width:=1280
+                                          depth_height:=720
+                                          depth_fps:=30
+                                          infra_width:=640
+                                          infra_height:=480
+                                          infra_fps:=30
+                                          color_width:=1920
+                                          color_height:=1080
+                                          color_fps:=30
+                                          *origin">
+    <xacro:property name="M_PI" value="3.1415926535897931"/>
+    <!-- The following values are approximate, and the camera node
+     publishing TF values with actual calibrated camera extrinsic values -->
+    <xacro:property name="d435i_cam_depth_to_left_ir_offset" value="0.0"/>
+    <xacro:property name="d435i_cam_depth_to_right_ir_offset" value="-0.050"/>
+    <xacro:property name="d435i_cam_depth_to_color_offset" value="0.015"/>
+    <!-- The following values model the aluminum peripherial case for the
+  	D435 camera, with the camera joint represented by the actual
+  	peripherial camera tripod mount -->
+    <xacro:property name="d435i_cam_width" value="0.090"/>
+    <xacro:property name="d435i_cam_height" value="0.025"/>
+    <xacro:property name="d435i_cam_depth" value="0.02505"/>
+    <xacro:property name="d435i_cam_mount_from_center_offset" value="0.0149"/>
+    <!-- The following offset is relative the the physical D435 camera peripherial
+  	camera tripod mount -->
+    <xacro:property name="d435i_cam_depth_px" value="${d435i_cam_mount_from_center_offset}"/>
+    <xacro:property name="d435i_cam_depth_py" value="0.0175"/>
+    <xacro:property name="d435i_cam_depth_pz" value="${d435i_cam_height/2}"/>
+    <material name="${name}_aluminum">
+	  <color rgba="0.5 0.5 0.5 1"/>
+    </material>
+    <!-- camera body, with origin at bottom screw mount -->
+    <joint name="${name}_joint" type="fixed">
+      <xacro:insert_block name="origin"/>
+      <parent link="${parent}"/>
+      <child link="${name}_bottom_screw_frame"/>
+    </joint>
+    <link name="${name}_bottom_screw_frame"/>
+    <joint name="${name}_link_joint" type="fixed">
+      <origin xyz="0 ${d435i_cam_depth_py} ${d435i_cam_depth_pz}" rpy="0 0 0"/>
+      <parent link="${name}_bottom_screw_frame"/>
+      <child link="${name}_link"/>
+    </joint>
+    <link name="${name}_link">
+      <visual>
+      <origin xyz="${d435i_cam_mount_from_center_offset} ${-d435i_cam_depth_py} 0" rpy="${M_PI/2} 0 ${M_PI/2}"/>
+        <geometry>
+          <!-- <box size="${d435i_cam_width} ${d435i_cam_height} ${d435i_cam_depth}"/> -->
+          <mesh filename="package://realsense2_description/meshes/d435.dae"/>
+          <!--<mesh filename="package://realsense2_description/meshes/d435/d435.dae"/>-->
+        </geometry>
+        <material name="${name}_aluminum"/>
+      </visual>
+      <collision>
+        <origin xyz="0 ${-d435i_cam_depth_py} 0" rpy="0 0 0"/>
+        <geometry>
+        <box size="${d435i_cam_depth} ${d435i_cam_width} ${d435i_cam_height}"/>
+        </geometry>
+      </collision>
+      <inertial>
+        <!-- The following are not reliable values, and should not be used for modeling -->
+        <mass value="0.564"/>
+        <origin xyz="0 0 0"/>
+        <inertia ixx="0.003881243" ixy="0.0" ixz="0.0" iyy="0.000498940" iyz="0.0" izz="0.003879257"/>
+      </inertial>
+    </link>
+    <!-- camera depth joints and links -->
+    <joint name="${name}_depth_joint" type="fixed">
+      <origin xyz="0 0 0" rpy="0 0 0"/>
+      <parent link="${name}_link"/>
+      <child link="${name}_depth_frame"/>
+    </joint>
+    <link name="${name}_depth_frame"/>
+    <joint name="${name}_depth_optical_joint" type="fixed">
+      <origin xyz="0 0 0" rpy="${-M_PI/2} 0 ${-M_PI/2}"/>
+      <parent link="${name}_depth_frame"/>
+      <child link="${name}_depth_optical_frame"/>
+    </joint>
+    <link name="${name}_depth_optical_frame"/>
+    <!-- camera left IR joints and links -->
+    <joint name="${name}_left_ir_joint" type="fixed">
+      <origin xyz="0 ${d435i_cam_depth_to_left_ir_offset} 0" rpy="0 0 0"/>
+      <parent link="${name}_depth_frame"/>
+      <child link="${name}_left_ir_frame"/>
+    </joint>
+    <link name="${name}_left_ir_frame"/>
+    <joint name="${name}_left_ir_optical_joint" type="fixed">
+      <origin xyz="0 0 0" rpy="${-M_PI/2} 0 ${-M_PI/2}"/>
+      <parent link="${name}_left_ir_frame"/>
+      <child link="${name}_left_ir_optical_frame"/>
+    </joint>
+    <link name="${name}_left_ir_optical_frame"/>
+    <!-- camera right IR joints and links -->
+    <joint name="${name}_right_ir_joint" type="fixed">
+      <origin xyz="0 ${d435i_cam_depth_to_right_ir_offset} 0" rpy="0 0 0"/>
+      <parent link="${name}_depth_frame"/>
+      <child link="${name}_right_ir_frame"/>
+    </joint>
+    <link name="${name}_right_ir_frame"/>
+    <joint name="${name}_right_ir_optical_joint" type="fixed">
+      <origin xyz="0 0 0" rpy="${-M_PI/2} 0 ${-M_PI/2}"/>
+      <parent link="${name}_right_ir_frame"/>
+      <child link="${name}_right_ir_optical_frame"/>
+    </joint>
+    <link name="${name}_right_ir_optical_frame"/>
+    <!-- camera color joints and links -->
+    <joint name="${name}_color_joint" type="fixed">
+      <origin xyz="0 ${d435i_cam_depth_to_color_offset} 0" rpy="0 0 0"/>
+      <parent link="${name}_depth_frame"/>
+      <child link="${name}_color_frame"/>
+    </joint>
+    <link name="${name}_color_frame"/>
+    <joint name="${name}_color_optical_joint" type="fixed">
+      <origin xyz="0 0 0" rpy="${-M_PI/2} 0 ${-M_PI/2}"/>
+      <parent link="${name}_color_frame"/>
+      <child link="${name}_color_optical_frame"/>
+    </joint>
+    <link name="${name}_color_optical_frame"/>
+    <!-- camera accel joints and links -->
+    <joint name="${name}_accel_joint" type="fixed">
+      <origin xyz="-0.00174 0.00552 0.0176" rpy="0 0 0"/>
+      <parent link="${name}_link"/>
+      <child link="${name}_accel_frame"/>
+    </joint>
+    <link name="${name}_accel_frame"/>
+    <joint name="${name}_accel_optical_joint" type="fixed">
+      <origin xyz="0 0 0" rpy="${-M_PI/2} 0 ${-M_PI/2}"/>
+      <parent link="${name}_accel_frame"/>
+      <child link="${name}_accel_optical_frame"/>
+    </joint>
+    <link name="${name}_accel_optical_frame"/>
+    <!-- camera gyro joints and links -->
+    <joint name="${name}_gyro_joint" type="fixed">
+      <origin xyz="-0.00174 0.00552 0.0176" rpy="0 0 0"/>
+      <parent link="${name}_link"/>
+      <child link="${name}_gyro_frame"/>
+    </joint>
+    <link name="${name}_gyro_frame"/>
+    <joint name="${name}_gyro_optical_joint" type="fixed">
+      <origin xyz="0 0 0" rpy="${-M_PI/2} 0 ${-M_PI/2}"/>
+      <parent link="${name}_gyro_frame"/>
+      <child link="${name}_gyro_optical_frame"/>
+    </joint>
+    <link name="${name}_gyro_optical_frame"/>
+    <!-- Realsense Gazebo Plugin -->
+    <xacro:gazebo_d435i camera_name="${name}"
+                        topics_ns="${topics_ns}"
+                        reference_link="${name}_link"
+                        depth_optical_frame="${name}_depth_optical_frame"
+                        depth_width="${depth_width}"
+                        depth_height="${depth_height}"
+                        depth_fps="${depth_fps}"
+                        color_optical_frame="${name}_color_optical_frame"
+                        color_width="${color_width}"
+                        color_height="${color_height}"
+                        color_fps="${color_fps}"
+                        infrared1_optical_frame="${name}_left_ir_optical_frame"
+                        infrared2_optical_frame="${name}_right_ir_optical_frame"
+                        infra_width="${infra_width}"
+                        infra_height="${infra_height}"
+                        infra_fps="${infra_fps}"
+                        accel_optical_frame="${name}_accel_optical_frame"
+                        gyro_optical_frame="${name}_gyro_optical_frame"
+                        accel_fps="${accel_fps}"
+                        gyro_fps="${gyro_fps}"
+                        enable_pointCloud="${enable_pointCloud}"
+                        unite_imu_method="${unite_imu_method}"
+                        clip_distance="${clip_distance}"
+                        align_depth="${align_depth}"
+                        visualize="${visualize}"
+    />
   </xacro:macro>
 </robot>
