Commit message: add cmakelist and package

File: urdf/turtlebot3_waffle_pi.urdf.xacro (robot description, xacro)
@@ -1,6 +1,6 @@
 <?xml version="1.0" ?>
 <robot name="turtlebot3_waffle_pi" xmlns:xacro="http://ros.org/wiki/xacro">
-  <xacro:include filename="$(find turtlebot3_description)/urdf/common_properties.xacro"/>
-  <xacro:include filename="$(find turtlebot3_description)/urdf/turtlebot3_waffle_pi.gazebo.xacro"/>
+  <xacro:include filename="$(find mai_sim)/urdf/common_properties.xacro"/>
+  <xacro:include filename="$(find mai_sim)/urdf/turtlebot3_waffle_pi.gazebo.xacro"/>
   <link name="base_footprint"/>
   <joint name="base_joint" type="fixed">
@@ -13,5 +13,5 @@
       <origin xyz="-0.064 0 0.0" rpy="0 0 0"/>
       <geometry>
-        <mesh filename="package://turtlebot3_description/meshes/bases/waffle_pi_base.stl" scale="0.001 0.001 0.001"/>
+        <mesh filename="package://mai_sim/meshes/bases/waffle_pi_base.stl" scale="0.001 0.001 0.001"/>
       </geometry>
       <material name="light_black"/>
@@ -41,5 +41,5 @@
       <origin xyz="0 0 0" rpy="1.57 0 0"/>
       <geometry>
-        <mesh filename="package://turtlebot3_description/meshes/wheels/left_tire.stl" scale="0.001 0.001 0.001"/>
+        <mesh filename="package://mai_sim/meshes/wheels/left_tire.stl" scale="0.001 0.001 0.001"/>
       </geometry>
       <material name="dark"/>
@@ -69,5 +69,5 @@
       <origin xyz="0 0 0" rpy="1.57 0 0"/>
       <geometry>
-        <mesh filename="package://turtlebot3_description/meshes/wheels/right_tire.stl" scale="0.001 0.001 0.001"/>
+        <mesh filename="package://mai_sim/meshes/wheels/right_tire.stl" scale="0.001 0.001 0.001"/>
       </geometry>
       <material name="dark"/>
@@ -142,5 +142,5 @@
       <origin xyz="0 0 0.0" rpy="0 0 0"/>
       <geometry>
-        <mesh filename="package://turtlebot3_description/meshes/sensors/lds.stl" scale="0.001 0.001 0.001"/>
+        <mesh filename="package://mai_sim/meshes/sensors/lds.stl" scale="0.001 0.001 0.001"/>
       </geometry>
       <material name="dark"/>

Commit message: add camera

File: urdf/turtlebot3_waffle_pi.urdf.xacro (robot description, xacro)
@@ -186,7 +186,7 @@
   <link name="camera_rgb_optical_frame"/> -->
   <!-- d435i frame definition can be found at https://github.com/IntelRealSense/librealsense/blob/master/doc/d435i.md -->
-  <xacro:include filename="$(find mai_sim)/urdf/_d435i.urdf.xacro"/>
-  <xacro:sensor_d435i parent="base_link" name="D435i_camera" topics_ns="D435i_camera">
-    <origin xyz="0.0 0.5 0.1" rpy="0.0 0.0 0.0"/>
-  </xacro:sensor_d435i>
+  <xacro:include filename="$(find mai_sim)/urdf/_d435.urdf.xacro"/>
+  <xacro:sensor_d435 parent="base_link" name="D435_camera" topics_ns="D435_camera">
+    <origin xyz="0.0 0.0 0.2" rpy="0.0 0.0 0.0"/>
+  </xacro:sensor_d435>
 </robot>

Commit message: rtabmap work

File: urdf/turtlebot3_waffle_pi.urdf.xacro (robot description, xacro)
@@ -186,7 +186,15 @@
   <link name="camera_rgb_optical_frame"/> -->
   <!-- d435i frame definition can be found at https://github.com/IntelRealSense/librealsense/blob/master/doc/d435i.md -->
-  <xacro:include filename="$(find mai_sim)/urdf/_d435.urdf.xacro"/>
+  <!-- <xacro:include filename="$(find mai_sim)/urdf/_d435.urdf.xacro"/>
   <xacro:sensor_d435 parent="base_link" name="camera" topics_ns="D435_camera" publish_pointcloud="true">
     <origin xyz="0.0 0.0 0.2" rpy="0.0 0.0 0.0"/>
-  </xacro:sensor_d435>
+  </xacro:sensor_d435> -->
+  <xacro:arg name="use_nominal_extrinsics" default="false" />
+  <xacro:include filename="$(find realsense2_description)/urdf/_d435i.urdf.xacro"/>
+  <xacro:sensor_d435i parent="base_link" name="camera1" use_nominal_extrinsics="$(arg use_nominal_extrinsics)">
+    <origin xyz="0 0.05 0.2" rpy="0.0 0.0 1.57079633"/>
+  </xacro:sensor_d435i>
+  <xacro:sensor_d435i parent="base_link" name="camera2" use_nominal_extrinsics="$(arg use_nominal_extrinsics)">
+    <origin xyz="0.0 -0.05 0.2" rpy="0.0 0.0 -1.57079633"/>
+  </xacro:sensor_d435i>
 </robot>
